Commit message: continue rgb projection

File: launch/include/config/robot.urdf.xacro (robot description, xacro)
@@ -21,4 +21,10 @@
     <origin xyz="0 0 0" rpy="0 0 0" />
   </joint>
+  <!-- <link name="camera"> </link>
+  <joint name="camera_joint" type="fixed">
+    <parent link="chassis_link" />
+    <child link="stereo" />
+    <origin xyz="0.0911526 0.0954019 -0.187078" rpy="-1.69052 0.00123675 -1.58841" />
+  </joint> -->
   <link name="navsat_link"> </link>
   <joint name="navsat_joint" type="fixed">

Commit message: finished rgb projection

File: launch/include/config/robot.urdf.xacro (robot description, xacro)
@@ -21,10 +21,4 @@
     <origin xyz="0 0 0" rpy="0 0 0" />
   </joint>
-  <!-- <link name="camera"> </link>
-  <joint name="camera_joint" type="fixed">
-    <parent link="chassis_link" />
-    <child link="stereo" />
-    <origin xyz="0.0911526 0.0954019 -0.187078" rpy="-1.69052 0.00123675 -1.58841" />
-  </joint> -->
   <link name="navsat_link"> </link>
   <joint name="navsat_joint" type="fixed">
